Commit message: Update RViz config and fix TF timestamp issue

File: ros2_ws/src/amr_description_pkg/urdf/amr.urdf.xacro (robot description, xacro)
@@ -2,20 +2,21 @@
 <robot name="vehicle_blue" xmlns:xacro="http://ros.org/wiki/xacro">
   <!-- Define robot constants -->
-  <xacro:property name="base_width" value="1.0"/>
-  <xacro:property name="base_length" value="2.0"/>
-  <xacro:property name="base_height" value="0.5"/>
-  <xacro:property name="wheel_radius" value="0.4"/>
-  <xacro:property name="wheel_width" value="0.2"/>
-  <xacro:property name="wheel_ygap" value="0.1"/> <!-- Gap between chassis and wheel -->
-  <xacro:property name="wheel_zoff" value="0.0"/> <!-- Wheel z offset -->
-  <xacro:property name="wheel_xoff" value="0.5"/> <!-- Wheel x offset from center (rear) -->
-  <xacro:property name="caster_xoff" value="0.8"/> <!-- Caster x offset (front) -->
-  <xacro:property name="caster_radius" value="0.2"/>
+  <xacro:property name="base_width" value="1.0" />
+  <xacro:property name="base_length" value="2.0" />
+  <xacro:property name="base_height" value="0.5" />
+  <xacro:property name="wheel_radius" value="0.4" />
+  <xacro:property name="wheel_width" value="0.2" />
+  <xacro:property name="wheel_ygap" value="0.1" /> <!-- Gap between chassis and wheel -->
+  <xacro:property name="wheel_zoff" value="0.0" /> <!-- Wheel z offset -->
+  <xacro:property name="wheel_xoff" value="0.5" /> <!-- Wheel x offset from center (rear) -->
+  <xacro:property name="caster_xoff" value="0.8" /> <!-- Caster x offset (front) -->
+  <xacro:property name="caster_radius" value="0.2" />
   <!-- Define intertial property macros  -->
   <xacro:macro name="box_inertia" params="m w h d">
     <inertial>
-      <origin xyz="0 0 0" rpy="${pi/2} 0 ${pi/2}"/>
-      <mass value="${m}"/>
-      <inertia ixx="${(m/12) * (h*h + d*d)}" ixy="0.0" ixz="0.0" iyy="${(m/12) * (w*w + d*d)}" iyz="0.0" izz="${(m/12) * (w*w + h*h)}"/>
+      <origin xyz="0 0 0" rpy="${pi/2} 0 ${pi/2}" />
+      <mass value="${m}" />
+      <inertia ixx="${(m/12) * (h*h + d*d)}" ixy="0.0" ixz="0.0" iyy="${(m/12) * (w*w + d*d)}"
+        iyz="0.0" izz="${(m/12) * (w*w + h*h)}" />
     </inertial>
   </xacro:macro>
@@ -23,12 +24,14 @@
     <inertial>
       <origin xyz="0 0 0" rpy="${pi/2} 0 0" />
-      <mass value="${m}"/>
-      <inertia ixx="${(m/12) * (3*r*r + h*h)}" ixy = "0" ixz = "0" iyy="${(m/12) * (3*r*r + h*h)}" iyz = "0" izz="${(m/2) * (r*r)}"/>
+      <mass value="${m}" />
+      <inertia ixx="${(m/12) * (3*r*r + h*h)}" ixy="0" ixz="0" iyy="${(m/12) * (3*r*r + h*h)}"
+        iyz="0" izz="${(m/2) * (r*r)}" />
     </inertial>
   </xacro:macro>
   <xacro:macro name="sphere_inertia" params="m r">
     <inertial>
-      <mass value="${m}"/>
-      <inertia ixx="${(2/5) * m * (r*r)}" ixy="0.0" ixz="0.0" iyy="${(2/5) * m * (r*r)}" iyz="0.0" izz="${(2/5) * m * (r*r)}"/>
+      <mass value="${m}" />
+      <inertia ixx="${(2/5) * m * (r*r)}" ixy="0.0" ixz="0.0" iyy="${(2/5) * m * (r*r)}" iyz="0.0"
+        izz="${(2/5) * m * (r*r)}" />
     </inertial>
   </xacro:macro>
@@ -39,21 +42,21 @@
     <visual>
       <geometry>
-        <box size="${base_length} ${base_width} ${base_height}"/>
+        <box size="${base_length} ${base_width} ${base_height}" />
       </geometry>
       <material name="Blue">
-        <color rgba="0 0 1.0 1.0"/>
+        <color rgba="0 0 1.0 1.0" />
       </material>
     </visual>
     <collision>
       <geometry>
-        <box size="${base_length} ${base_width} ${base_height}"/>
+        <box size="${base_length} ${base_width} ${base_height}" />
       </geometry>
     </collision>
-    <xacro:box_inertia m="15" w="${base_width}" d="${base_length}" h="${base_height}"/>
+    <xacro:box_inertia m="15" w="${base_width}" d="${base_length}" h="${base_height}" />
   </link>
   <joint name="base_joint" type="fixed">
-    <parent link="base_link"/>
-    <child link="chassis"/>
-    <origin xyz="0.0 0.0 ${wheel_radius}" rpy="0 0 0"/>
+    <parent link="chassis" />
+    <child link="base_link" />
+    <origin xyz="0.0 0.0 -${wheel_radius}" rpy="0 0 0" />
   </joint>
   <!-- Wheels -->
@@ -61,25 +64,26 @@
     <link name="${prefix}_link">
       <visual>
-        <origin xyz="0 0 0" rpy="${pi/2} 0 0"/>
+        <origin xyz="0 0 0" rpy="${pi/2} 0 0" />
         <geometry>
-            <cylinder radius="${wheel_radius}" length="${wheel_width}"/>
+          <cylinder radius="${wheel_radius}" length="${wheel_width}" />
         </geometry>
         <material name="Red">
-          <color rgba="1.0 0 0 1.0"/>
+          <color rgba="1.0 0 0 1.0" />
         </material>
       </visual>
       <collision>
-        <origin xyz="0 0 0" rpy="${pi/2} 0 0"/>
+        <origin xyz="0 0 0" rpy="${pi/2} 0 0" />
         <geometry>
-          <cylinder radius="${wheel_radius}" length="${wheel_width}"/>
+          <cylinder radius="${wheel_radius}" length="${wheel_width}" />
         </geometry>
       </collision>
-      <xacro:cylinder_inertia m="0.5" r="${wheel_radius}" h="${wheel_width}"/>
+      <xacro:cylinder_inertia m="0.5" r="${wheel_radius}" h="${wheel_width}" />
     </link>
     <joint name="${prefix}_joint" type="continuous">
-      <parent link="chassis"/>
-      <child link="${prefix}_link"/>
-      <origin xyz="${-wheel_xoff} ${y_reflect*(base_width/2 + wheel_ygap)} ${-wheel_zoff}" rpy="0 0 0"/>
-      <axis xyz="0 1 0"/>
+      <parent link="chassis" />
+      <child link="${prefix}_link" />
+      <origin xyz="${-wheel_xoff} ${y_reflect*(base_width/2 + wheel_ygap)} ${-wheel_zoff}"
+        rpy="0 0 0" />
+      <axis xyz="0 1 0" />
     </joint>
   </xacro:macro>
@@ -90,21 +94,21 @@
     <visual>
       <geometry>
-        <sphere radius="${caster_radius}"/>
+        <sphere radius="${caster_radius}" />
       </geometry>
       <material name="Green">
-        <color rgba="0 1.0 0 1.0"/>
+        <color rgba="0 1.0 0 1.0" />
       </material>
     </visual>
     <collision>
       <geometry>
-        <sphere radius="${caster_radius}"/>
+        <sphere radius="${caster_radius}" />
       </geometry>
     </collision>
-    <xacro:sphere_inertia m="0.5" r="${caster_radius}"/>
+    <xacro:sphere_inertia m="0.5" r="${caster_radius}" />
   </link>
   <joint name="caster_joint" type="fixed">
-    <parent link="chassis"/>
-    <child link="caster"/>
-    <origin xyz="${caster_xoff} 0.0 ${-(base_height/2)}" rpy="0 0 0"/>
+    <parent link="chassis" />
+    <child link="caster" />
+    <origin xyz="${caster_xoff} 0.0 ${-(base_height/2)}" rpy="0 0 0" />
   </joint>
   <!-- IMU -->
@@ -112,15 +116,15 @@
     <visual>
       <geometry>
-        <box size="0.1 0.1 0.1"/>
+        <box size="0.1 0.1 0.1" />
       </geometry>
       <material name="Black">
-        <color rgba="0 0 0 1.0"/>
+        <color rgba="0 0 0 1.0" />
       </material>
     </visual>
   </link>
   <joint name="imu_joint" type="fixed">
-    <parent link="chassis"/>
-    <child link="imu_link"/>
-    <origin xyz="0 0 0" rpy="0 0 0"/>
+    <parent link="chassis" />
+    <child link="imu_link" />
+    <origin xyz="0 0 0" rpy="0 0 0" />
   </joint>
   <!-- LiDAR -->
@@ -128,15 +132,15 @@
     <visual>
       <geometry>
-        <cylinder radius="0.1" length="0.1"/>
+        <cylinder radius="0.1" length="0.1" />
       </geometry>
       <material name="Black">
-        <color rgba="0 0 0 1.0"/>
+        <color rgba="0 0 0 1.0" />
       </material>
     </visual>
   </link>
   <joint name="lidar_joint" type="fixed">
-    <parent link="chassis"/>
-    <child link="lidar_link"/>
-    <origin xyz="0.8 0 0.5" rpy="0 0 0"/>
+    <parent link="chassis" />
+    <child link="lidar_link" />
+    <origin xyz="0.8 0 0.5" rpy="0 0 0" />
   </joint>
 </robot>

Commit message: Fix TF issues: Invert base_joint, update SDF frames, adjust launch file

File: ros2_ws/src/amr_description_pkg/urdf/amr.urdf.xacro (robot description, xacro)
@@ -56,7 +56,7 @@
   </link>
   <joint name="base_joint" type="fixed">
-    <parent link="chassis" />
-    <child link="base_link" />
-    <origin xyz="0.0 0.0 -${wheel_radius}" rpy="0 0 0" />
+    <parent link="base_link" />
+    <child link="chassis" />
+    <origin xyz="0.0 0.0 ${wheel_radius}" rpy="0 0 0" />
   </joint>
   <!-- Wheels -->

Commit message: Update robot shape: lower chassis, center wheels, add rear caster, fix collision

File: ros2_ws/src/amr_description_pkg/urdf/amr.urdf.xacro (robot description, xacro)
@@ -2,14 +2,14 @@
 <robot name="vehicle_blue" xmlns:xacro="http://ros.org/wiki/xacro">
   <!-- Define robot constants -->
-  <xacro:property name="base_width" value="1.0" />
-  <xacro:property name="base_length" value="2.0" />
-  <xacro:property name="base_height" value="0.5" />
-  <xacro:property name="wheel_radius" value="0.4" />
-  <xacro:property name="wheel_width" value="0.2" />
+  <xacro:property name="base_width" value="0.6" />
+  <xacro:property name="base_length" value="1.0" />
+  <xacro:property name="base_height" value="0.2" />
+  <xacro:property name="wheel_radius" value="0.15" />
+  <xacro:property name="wheel_width" value="0.1" />
   <xacro:property name="wheel_ygap" value="0.1" /> <!-- Gap between chassis and wheel -->
-  <xacro:property name="wheel_zoff" value="0.0" /> <!-- Wheel z offset -->
-  <xacro:property name="wheel_xoff" value="0.5" /> <!-- Wheel x offset from center (rear) -->
-  <xacro:property name="caster_xoff" value="0.8" /> <!-- Caster x offset (front) -->
-  <xacro:property name="caster_radius" value="0.2" />
+  <xacro:property name="wheel_zoff" value="0.15" /> <!-- Wheel z offset -->
+  <xacro:property name="wheel_xoff" value="0.0" /> <!-- Wheel x offset from center (rear) -->
+  <xacro:property name="caster_xoff" value="0.4" /> <!-- Caster x offset (front) -->
+  <xacro:property name="caster_radius" value="0.05" />
   <!-- Define intertial property macros  -->
   <xacro:macro name="box_inertia" params="m w h d">
@@ -53,10 +53,10 @@
       </geometry>
     </collision>
-    <xacro:box_inertia m="15" w="${base_width}" d="${base_length}" h="${base_height}" />
+    <xacro:box_inertia m="30" w="${base_width}" d="${base_length}" h="${base_height}" />
   </link>
   <joint name="base_joint" type="fixed">
     <parent link="base_link" />
     <child link="chassis" />
-    <origin xyz="0.0 0.0 ${wheel_radius}" rpy="0 0 0" />
+    <origin xyz="0.0 0.0 0.2" rpy="0 0 0" />
   </joint>
   <!-- Wheels -->
@@ -90,6 +90,6 @@
   <xacro:wheel prefix="left_wheel" x_reflect="-1" y_reflect="1" />
   <xacro:wheel prefix="right_wheel" x_reflect="-1" y_reflect="-1" />
-  <!-- Caster Wheel -->
-  <link name="caster">
+  <!-- Front Caster Wheel -->
+  <link name="front_caster">
     <visual>
       <geometry>
@@ -107,8 +107,30 @@
     <xacro:sphere_inertia m="0.5" r="${caster_radius}" />
   </link>
-  <joint name="caster_joint" type="fixed">
+  <joint name="front_caster_joint" type="fixed">
     <parent link="chassis" />
-    <child link="caster" />
-    <origin xyz="${caster_xoff} 0.0 ${-(base_height/2)}" rpy="0 0 0" />
+    <child link="front_caster" />
+    <origin xyz="${caster_xoff} 0.0 -0.15" rpy="0 0 0" />
+  </joint>
+  <!-- Rear Caster Wheel -->
+  <link name="rear_caster">
+    <visual>
+      <geometry>
+        <sphere radius="${caster_radius}" />
+      </geometry>
+      <material name="Green">
+        <color rgba="0 1.0 0 1.0" />
+      </material>
+    </visual>
+    <collision>
+      <geometry>
+        <sphere radius="${caster_radius}" />
+      </geometry>
+    </collision>
+    <xacro:sphere_inertia m="0.5" r="${caster_radius}" />
+  </link>
+  <joint name="rear_caster_joint" type="fixed">
+    <parent link="chassis" />
+    <child link="rear_caster" />
+    <origin xyz="${-caster_xoff} 0.0 -0.15" rpy="0 0 0" />
   </joint>
   <!-- IMU -->
@@ -142,5 +164,5 @@
     <parent link="chassis" />
     <child link="lidar_link" />
-    <origin xyz="0.8 0 0.5" rpy="0 0 0" />
+    <origin xyz="0.4 0 0.2" rpy="0 0 0" />
   </joint>
 </robot>
