Commit message: Backup before revert

File: ros2_ws/src/amr_description/urdf/amr.urdf.xacro (robot description, xacro)
@@ -37,7 +37,12 @@
   </xacro:macro>
   <!-- Robot Base -->
+  <link name="base_footprint">
+  </link>
+  <joint name="base_joint" type="fixed">
+    <parent link="base_footprint" />
+    <child link="base_link" />
+    <origin xyz="0.0 0.0 0.2" rpy="0 0 0" />
+  </joint>
   <link name="base_link">
-  </link>
-  <link name="chassis">
     <visual>
       <geometry>
@@ -55,9 +60,4 @@
     <xacro:box_inertia m="30" w="${base_width}" d="${base_length}" h="${base_height}" />
   </link>
-  <joint name="base_joint" type="fixed">
-    <parent link="base_link" />
-    <child link="chassis" />
-    <origin xyz="0.0 0.0 0.2" rpy="0 0 0" />
-  </joint>
   <!-- Wheels -->
   <xacro:macro name="wheel" params="prefix x_reflect y_reflect">
@@ -81,5 +81,5 @@
     </link>
     <joint name="${prefix}_joint" type="continuous">
-      <parent link="chassis" />
+      <parent link="base_link" />
       <child link="${prefix}_link" />
       <origin xyz="${-wheel_xoff} ${y_reflect*(base_width/2 + wheel_ygap)} ${-wheel_zoff}"
@@ -108,5 +108,5 @@
   </link>
   <joint name="front_caster_joint" type="fixed">
-    <parent link="chassis" />
+    <parent link="base_link" />
     <child link="front_caster" />
     <origin xyz="${caster_xoff} 0.0 -0.15" rpy="0 0 0" />
@@ -130,5 +130,5 @@
   </link>
   <joint name="rear_caster_joint" type="fixed">
-    <parent link="chassis" />
+    <parent link="base_link" />
     <child link="rear_caster" />
     <origin xyz="${-caster_xoff} 0.0 -0.15" rpy="0 0 0" />
@@ -146,5 +146,5 @@
   </link>
   <joint name="imu_joint" type="fixed">
-    <parent link="chassis" />
+    <parent link="base_link" />
     <child link="imu_link" />
     <origin xyz="0 0 0" rpy="0 0 0" />
@@ -162,5 +162,5 @@
   </link>
   <joint name="lidar_joint" type="fixed">
-    <parent link="chassis" />
+    <parent link="base_link" />
     <child link="lidar_link" />
     <origin xyz="0.4 0 0.2" rpy="0 0 0" />

Commit message: Implement SLAM, expand world, and fix time jumps

File: ros2_ws/src/amr_description/urdf/amr.urdf.xacro (robot description, xacro)
@@ -11,5 +11,5 @@
   <xacro:property name="wheel_xoff" value="0.0" /> <!-- Wheel x offset from center (rear) -->
   <xacro:property name="caster_xoff" value="0.4" /> <!-- Caster x offset (front) -->
-  <xacro:property name="caster_radius" value="0.05" />
+  <xacro:property name="caster_radius" value="0.15" />
   <!-- Define intertial property macros  -->
   <xacro:macro name="box_inertia" params="m w h d">

Commit message: Update robot model: reduce wheel/caster size, base height, and wheel separation

File: ros2_ws/src/amr_description/urdf/amr.urdf.xacro (robot description, xacro)
@@ -4,12 +4,12 @@
   <xacro:property name="base_width" value="0.6" />
   <xacro:property name="base_length" value="1.0" />
-  <xacro:property name="base_height" value="0.2" />
-  <xacro:property name="wheel_radius" value="0.15" />
+  <xacro:property name="base_height" value="0.1" />
+  <xacro:property name="wheel_radius" value="0.075" />
   <xacro:property name="wheel_width" value="0.1" />
-  <xacro:property name="wheel_ygap" value="0.1" /> <!-- Gap between chassis and wheel -->
-  <xacro:property name="wheel_zoff" value="0.15" /> <!-- Wheel z offset -->
+  <xacro:property name="wheel_ygap" value="-0.05" /> <!-- Gap between chassis and wheel -->
+  <xacro:property name="wheel_zoff" value="0.075" /> <!-- Wheel z offset -->
   <xacro:property name="wheel_xoff" value="0.0" /> <!-- Wheel x offset from center (rear) -->
   <xacro:property name="caster_xoff" value="0.4" /> <!-- Caster x offset (front) -->
-  <xacro:property name="caster_radius" value="0.15" />
+  <xacro:property name="caster_radius" value="0.075" />
   <!-- Define intertial property macros  -->
   <xacro:macro name="box_inertia" params="m w h d">
@@ -42,5 +42,5 @@
     <parent link="base_footprint" />
     <child link="base_link" />
-    <origin xyz="0.0 0.0 0.2" rpy="0 0 0" />
+    <origin xyz="0.0 0.0 0.15" rpy="0 0 0" />
   </joint>
   <link name="base_link">
@@ -110,5 +110,5 @@
     <parent link="base_link" />
     <child link="front_caster" />
-    <origin xyz="${caster_xoff} 0.0 -0.15" rpy="0 0 0" />
+    <origin xyz="${caster_xoff} 0.0 -0.075" rpy="0 0 0" />
   </joint>
   <!-- Rear Caster Wheel -->
@@ -132,5 +132,5 @@
     <parent link="base_link" />
     <child link="rear_caster" />
-    <origin xyz="${-caster_xoff} 0.0 -0.15" rpy="0 0 0" />
+    <origin xyz="${-caster_xoff} 0.0 -0.075" rpy="0 0 0" />
   </joint>
   <!-- IMU -->
@@ -164,5 +164,5 @@
     <parent link="base_link" />
     <child link="lidar_link" />
-    <origin xyz="0.4 0 0.2" rpy="0 0 0" />
+    <origin xyz="0.4 0 0.1" rpy="0 0 0" />
   </joint>
 </robot>
